File: hardware/plaquita_z80/z80.brd (EAGLE design)
At the start: 34.3 x 24.5 mm, 12 parts, among them U2 REG1117

Commit message: git-svn-id: http://www.atc.us.es/svn/zxuno@1325 c9f0b58d-52e7-4fa3-91d2-c85e4586ca94
Connections:
- removed net A17: IC1.31, J11.6
- removed net A18: IC1.29, J12.5
- removed net A20: IC1.34, J10.4
- new net A11: IC1.40, J11.3
- new net A12: IC1.41, J10.2
- new net A13: IC1.42, J12.2
- net A0: now also IC1.27, J10.6; no longer IC1.44, J10.1
- net A15: now also IC1.44, J10.1; no longer IC1.27, J10.6
- net A2: now also IC1.29, J12.5; no longer IC1.42, J12.2
- net A3: now also IC1.30, J10.5; no longer IC1.41, J10.2
- net A4: now also IC1.31, J11.6; no longer IC1.40, J11.3
- net A5: now also IC1.32, J12.6; no longer IC1.30, J10.5
- net A6: now also IC1.34, J10.4; no longer IC1.32, J12.6
- net BUSACK: now also X1.3; no longer J10.8
- net BUSREQ: now also X1.1; no longer J12.10
- net CLK: now also J10.7
- net D0: now also J12.10; no longer X1.6
- net D1: now also J11.10; no longer X1.4
- net D2: now also J10.8; no longer X1.5
- net D7: now also J11.7; no longer X1.9
- net HALT: now also X1.4; no longer X1.1
- net INT: now also X1.9; no longer X1.3
- net NMI: now also X1.5; no longer X1.2
- net RESET: now also X1.6; no longer J10.7
- net RFSH: no longer J11.7
- net WAIT: now also X1.2; no longer J11.10
Routing:
- net GND: track 48.5 -> 76.6 mm, vias 2 -> 3
- net CLK: track 0.00 -> 22.9 mm, vias 0 -> 2
- net A12: track 0.00 -> 22.6 mm
- net A11: track 0.00 -> 18.6 mm
- net A13: track 0.00 -> 18.4 mm
- net D1: track 10.1 -> 25.7 mm, vias 0 -> 2
- net A15: track 13.6 -> 26.4 mm
- net A0: track 26.4 -> 13.6 mm
- net A20: track 12.6 -> 0.00 mm
- net A18: track 12.2 -> 0.00 mm
- net RFSH: track 11.8 -> 0.00 mm
- net A17: track 11.7 -> 0.00 mm
- net D7: track 11.9 -> 23.3 mm
- net D2: track 12.3 -> 22.9 mm, vias 0 -> 2
- net A5: track 16.0 -> 7.27 mm
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