File: hardware/plaquita_z80/z80.sch (EAGLE design)
At the start: 12 parts, among them U2 REG1117

Commit message: git-svn-id: http://www.atc.us.es/svn/zxuno@1325 c9f0b58d-52e7-4fa3-91d2-c85e4586ca94
Connections:
- removed net A17: IC1G$1.A4, J11.6
- removed net A18: IC1G$1.A2, J12.5
- removed net A20: IC1G$1.A6, J10.4
- new net A11: IC1G$1.A11, J11.3
- new net A12: IC1G$1.A12, J10.2
- new net A13: IC1G$1.A13, J12.2
- net A0: now also IC1G$1.A0, J10.6; no longer IC1G$1.A15, J10.1
- net A15: now also IC1G$1.A15, J10.1; no longer IC1G$1.A0, J10.6
- net A2: now also IC1G$1.A2, J12.5; no longer IC1G$1.A13, J12.2
- net A3: now also IC1G$1.A3, J10.5; no longer IC1G$1.A12, J10.2
- net A4: now also IC1G$1.A4, J11.6; no longer IC1G$1.A11, J11.3
- net A5: now also IC1G$1.A5, J12.6; no longer IC1G$1.A3, J10.5
- net A6: now also IC1G$1.A6, J10.4; no longer IC1G$1.A5, J12.6
- net BUSACK: now also X1.3; no longer J10.8
- net BUSREQ: now also X1.1; no longer J12.10
- net CLK: now also J10.7
- net D0: now also J12.10; no longer X1.6
- net D1: now also J11.10; no longer X1.4
- net D2: now also J10.8; no longer X1.5
- net D7: now also J11.7; no longer X1.9
- net HALT: now also X1.4; no longer X1.1
- net INT: now also X1.9; no longer X1.3
- net NMI: now also X1.5; no longer X1.2
- net RESET: now also X1.6; no longer J10.7
- net RFSH: no longer J11.7
- net WAIT: now also X1.2; no longer J11.10
Changed lines of the file:
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@@
 <?xml version="1.0" encoding="utf-8"?>
 <!DOCTYPE eagle SYSTEM "eagle.dtd">
-<eagle version="7.3.0">
+<eagle version="8.2.2">
 <drawing>
 <settings>
@@
 </segment>
 <segment>
-<wire x1="71.12" y1="99.06" x2="78.74" y2="99.06" width="0.1524" layer="91"/>
-<label x="76.2" y="99.06" size="1.778" layer="95"/>
-<pinref part="X1" gate="G$1" pin="9"/>
+<pinref part="J11" gate="G$1" pin="7"/>
+<wire x1="76.2" y1="68.58" x2="66.04" y2="68.58" width="0.1524" layer="91"/>
+<label x="66.04" y="68.58" size="1.778" layer="95"/>
 </segment>
 </net>
@@
 </segment>
 </net>
-<net name="A15" class="0">
+<net name="A0" class="0">
 <segment>
 <pinref part="IC1" gate="G$1" pin="A0"/>
@@
 </segment>
 </net>
-<net name="A0" class="0">
+<net name="A15" class="0">
 <segment>
 <pinref part="J10" gate="G$1" pin="1"/>
@@
 </segment>
 </net>
-<net name="A2" class="0">
+<net name="A13" class="0">
 <segment>
 <pinref part="J12" gate="G$1" pin="2"/>
@@
 </segment>
 </net>
-<net name="A3" class="0">
+<net name="A12" class="0">
 <segment>
 <pinref part="J10" gate="G$1" pin="2"/>
@@
 </segment>
 </net>
-<net name="A4" class="0">
+<net name="A11" class="0">
 <segment>
 <pinref part="J11" gate="G$1" pin="3"/>
@@
 </segment>
 </net>
-<net name="A5" class="0">
+<net name="A3" class="0">
 <segment>
 <pinref part="J10" gate="G$1" pin="5"/>
@@
 </segment>
 </net>
-<net name="A6" class="0">
+<net name="A5" class="0">
 <segment>
 <pinref part="J12" gate="G$1" pin="6"/>
@@
 </segment>
 </net>
-<net name="A17" class="0">
+<net name="A4" class="0">
 <segment>
 <pinref part="J11" gate="G$1" pin="6"/>
@@
 </segment>
 </net>
-<net name="A18" class="0">
+<net name="A2" class="0">
 <segment>
 <pinref part="J12" gate="G$1" pin="5"/>
@@
 </segment>
 </net>
-<net name="A20" class="0">
+<net name="A6" class="0">
 <segment>
 <pinref part="J10" gate="G$1" pin="4"/>
@@
 <pinref part="IC1" gate="G$1" pin="RFSH"/>
 </segment>
-<segment>
-<pinref part="J11" gate="G$1" pin="7"/>
-<wire x1="66.04" y1="68.58" x2="76.2" y2="68.58" width="0.1524" layer="91"/>
-<label x="66.04" y="68.58" size="1.778" layer="95"/>
-</segment>
 </net>
 <net name="HALT" class="0">
@@
 </segment>
 <segment>
-<wire x1="48.26" y1="109.22" x2="55.88" y2="109.22" width="0.1524" layer="91"/>
-<label x="48.26" y="109.22" size="1.778" layer="95"/>
-<pinref part="X1" gate="G$1" pin="1"/>
+<pinref part="X1" gate="G$1" pin="4"/>
+<wire x1="55.88" y1="101.6" x2="48.26" y2="101.6" width="0.1524" layer="91"/>
+<label x="48.26" y="101.6" size="1.778" layer="95"/>
 </segment>
 </net>
@@
 </segment>
 <segment>
-<pinref part="J11" gate="G$1" pin="10"/>
-<wire x1="66.04" y1="60.96" x2="76.2" y2="60.96" width="0.1524" layer="91"/>
-<label x="66.04" y="60.96" size="1.778" layer="95"/>
+<pinref part="X1" gate="G$1" pin="2"/>
+<wire x1="55.88" y1="106.68" x2="48.26" y2="106.68" width="0.1524" layer="91"/>
+<label x="48.26" y="106.68" size="1.778" layer="95"/>
 </segment>
 </net>
@@
 </segment>
 <segment>
-<wire x1="48.26" y1="104.14" x2="55.88" y2="104.14" width="0.1524" layer="91"/>
-<label x="48.26" y="104.14" size="1.778" layer="95"/>
-<pinref part="X1" gate="G$1" pin="3"/>
+<pinref part="X1" gate="G$1" pin="9"/>
+<wire x1="71.12" y1="99.06" x2="78.74" y2="99.06" width="0.1524" layer="91"/>
+<label x="76.2" y="99.06" size="1.778" layer="95"/>
 </segment>
 </net>
@@
 </segment>
 <segment>
-<wire x1="48.26" y1="106.68" x2="55.88" y2="106.68" width="0.1524" layer="91"/>
-<label x="48.26" y="106.68" size="1.778" layer="95"/>
-<pinref part="X1" gate="G$1" pin="2"/>
+<pinref part="X1" gate="G$1" pin="5"/>
+<wire x1="55.88" y1="99.06" x2="48.26" y2="99.06" width="0.1524" layer="91"/>
+<label x="48.26" y="99.06" size="1.778" layer="95"/>
 </segment>
 </net>
@@
 </segment>
 <segment>
+<pinref part="X1" gate="G$1" pin="6"/>
+<wire x1="71.12" y1="106.68" x2="78.74" y2="106.68" width="0.1524" layer="91"/>
+<label x="76.2" y="106.68" size="1.778" layer="95"/>
+</segment>
+</net>
+<net name="BUSREQ" class="0">
+<segment>
+<wire x1="-40.64" y1="50.8" x2="-33.02" y2="50.8" width="0.1524" layer="91"/>
+<label x="-40.64" y="50.8" size="1.778" layer="95"/>
+<pinref part="IC1" gate="G$1" pin="BUSREQ"/>
+</segment>
+<segment>
+<pinref part="X1" gate="G$1" pin="1"/>
+<wire x1="55.88" y1="109.22" x2="48.26" y2="109.22" width="0.1524" layer="91"/>
+<label x="48.26" y="109.22" size="1.778" layer="95"/>
+</segment>
+</net>
+<net name="BUSACK" class="0">
+<segment>
+<wire x1="-40.64" y1="48.26" x2="-33.02" y2="48.26" width="0.1524" layer="91"/>
+<label x="-40.64" y="48.26" size="1.778" layer="95"/>
+<pinref part="IC1" gate="G$1" pin="BUSACK"/>
+</segment>
+<segment>
+<pinref part="X1" gate="G$1" pin="3"/>
+<wire x1="55.88" y1="104.14" x2="48.26" y2="104.14" width="0.1524" layer="91"/>
+<label x="48.26" y="104.14" size="1.778" layer="95"/>
+</segment>
+</net>
+<net name="CLK" class="0">
+<segment>
+<wire x1="-40.64" y1="43.18" x2="-33.02" y2="43.18" width="0.1524" layer="91"/>
+<label x="-40.64" y="43.18" size="1.778" layer="95"/>
+<pinref part="IC1" gate="G$1" pin="CLK"/>
+</segment>
+<segment>
 <pinref part="J10" gate="G$1" pin="7"/>
 <wire x1="101.6" y1="68.58" x2="91.44" y2="68.58" width="0.1524" layer="91"/>
 <label x="91.44" y="68.58" size="1.778" layer="95"/>
-</segment>
-</net>
-<net name="BUSREQ" class="0">
-<segment>
-<wire x1="-40.64" y1="50.8" x2="-33.02" y2="50.8" width="0.1524" layer="91"/>
-<label x="-40.64" y="50.8" size="1.778" layer="95"/>
-<pinref part="IC1" gate="G$1" pin="BUSREQ"/>
-</segment>
-<segment>
-<pinref part="J12" gate="G$1" pin="10"/>
-<wire x1="38.1" y1="60.96" x2="48.26" y2="60.96" width="0.1524" layer="91"/>
-<label x="38.1" y="60.96" size="1.778" layer="95"/>
-</segment>
-</net>
-<net name="BUSACK" class="0">
-<segment>
-<wire x1="-40.64" y1="48.26" x2="-33.02" y2="48.26" width="0.1524" layer="91"/>
-<label x="-40.64" y="48.26" size="1.778" layer="95"/>
-<pinref part="IC1" gate="G$1" pin="BUSACK"/>
-</segment>
-<segment>
-<pinref part="J10" gate="G$1" pin="8"/>
-<wire x1="91.44" y1="66.04" x2="101.6" y2="66.04" width="0.1524" layer="91"/>
-<label x="91.44" y="66.04" size="1.778" layer="95"/>
-</segment>
-</net>
-<net name="CLK" class="0">
-<segment>
-<wire x1="-40.64" y1="43.18" x2="-33.02" y2="43.18" width="0.1524" layer="91"/>
-<label x="-40.64" y="43.18" size="1.778" layer="95"/>
-<pinref part="IC1" gate="G$1" pin="CLK"/>
 </segment>
 </net>
@@
 </segment>
 <segment>
-<wire x1="48.26" y1="99.06" x2="55.88" y2="99.06" width="0.1524" layer="91"/>
-<label x="48.26" y="99.06" size="1.778" layer="95"/>
-<pinref part="X1" gate="G$1" pin="5"/>
+<pinref part="J10" gate="G$1" pin="8"/>
+<wire x1="101.6" y1="66.04" x2="91.44" y2="66.04" width="0.1524" layer="91"/>
+<label x="91.44" y="66.04" size="1.778" layer="95"/>
 </segment>
 </net>
@@
 </segment>
 <segment>
-<wire x1="71.12" y1="106.68" x2="78.74" y2="106.68" width="0.1524" layer="91"/>
-<label x="76.2" y="106.68" size="1.778" layer="95"/>
-<pinref part="X1" gate="G$1" pin="6"/>
+<pinref part="J12" gate="G$1" pin="10"/>
+<wire x1="48.26" y1="60.96" x2="38.1" y2="60.96" width="0.1524" layer="91"/>
+<label x="38.1" y="60.96" size="1.778" layer="95"/>
 </segment>
 </net>
@@
 </segment>
 <segment>
-<wire x1="48.26" y1="101.6" x2="55.88" y2="101.6" width="0.1524" layer="91"/>
-<label x="48.26" y="101.6" size="1.778" layer="95"/>
-<pinref part="X1" gate="G$1" pin="4"/>
-</segment>
-</net>
+<pinref part="J11" gate="G$1" pin="10"/>
+<wire x1="76.2" y1="60.96" x2="66.04" y2="60.96" width="0.1524" layer="91"/>
+<label x="66.04" y="60.96" size="1.778" layer="95"/>
+</segment>
+</net>
